Commit message: REAL_ROBOT: real Franka Panda control + SpaceMouse teleop
- REAL_ROBOT/: scripts for real robot via franka_ros2
  - move_to_joint_angles.py: move to target joint angles with safety checks
  - real_robot_control.py: arm/gripper control, trajectory topic publish
  - spacemouse_control.py: SpaceMouse teleop (Joy -> IK -> joint commands)
  - README.md: setup, usage, SpaceMouse instructions
- SpaceMouse: position-only trajectory topic (no action), FK from real joints
- real_robot_control: get_current_arm_position(verbose), publish_joint_command topic-only

Co-authored-by: Cursor <cursoragent@cursor.com>

File: lerobot_teleoperator_devices/lerobot_teleoperator_devices/processors/_cache/panda_resolved.urdf (robot description, URDF)
Before this commit: robot panda, 12 links, 11 joints
Links:
- link panda_hand: geometry collision mesh filename=/home/cihan/lerobot-ros-agent/isaac_franka_moveit_perceptio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; visual mesh filename=/home/cihan/lerobot-ros-agent/isaac_franka_moveit_perceptio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
- link panda_leftfinger: geometry collision mesh filename=/home/cihan/lerobot-ros-agent/isaac_franka_moveit_perceptio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; visual mesh filename=/home/cihan/lerobot-ros-agent/isaac_franka_moveit_perceptio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
- link panda_link0: geometry collision mesh filename=/home/cihan/lerobot-ros-agent/isaac_franka_moveit_perceptio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; visual mesh filename=/home/cihan/lerobot-ros-agent/isaac_franka_moveit_perceptio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
- link panda_link1: geometry collision mesh filename=/home/cihan/lerobot-ros-agent/isaac_franka_moveit_perceptio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; visual mesh filename=/home/cihan/lerobot-ros-agent/isaac_franka_moveit_perceptio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
- link panda_link2: geometry collision mesh filename=/home/cihan/lerobot-ros-agent/isaac_franka_moveit_perceptio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; visual mesh filename=/home/cihan/lerobot-ros-agent/isaac_franka_moveit_perceptio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
- link panda_link3: geometry collision mesh filename=/home/cihan/lerobot-ros-agent/isaac_franka_moveit_perceptio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; visual mesh filename=/home/cihan/lerobot-ros-agent/isaac_franka_moveit_perceptio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
- link panda_link4: geometry collision mesh filename=/home/cihan/lerobot-ros-agent/isaac_franka_moveit_perceptio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; visual mesh filename=/home/cihan/lerobot-ros-agent/isaac_franka_moveit_perceptio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
- link panda_link5: geometry collision mesh filename=/home/cihan/lerobot-ros-agent/isaac_franka_moveit_perceptio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; visual mesh filename=/home/cihan/lerobot-ros-agent/isaac_franka_moveit_perceptio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
- link panda_link6: geometry collision mesh filename=/home/cihan/lerobot-ros-agent/isaac_franka_moveit_perceptio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; visual mesh filename=/home/cihan/lerobot-ros-agent/isaac_franka_moveit_perceptio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
- link panda_link7: geometry collision mesh filename=/home/cihan/lerobot-ros-agent/isaac_franka_moveit_perceptio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; visual mesh filename=/home/cihan/lerobot-ros-agent/isaac_franka_moveit_perceptio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
- link panda_rightfinger: geometry collision mesh filename=/home/cihan/lerobot-ros-agent/isaac_franka_moveit_perceptio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; visual mesh filename=/home/cihan/lerobot-ros-agent/isaac_franka_moveit_perceptio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
