Commit message: Add Polymetis-based data collection workflow and integrate new teleoperation updates.
This captures the current branch state with camera/recording script improvements, ROS teleoperator refinements, and policy/workflow reorganization so the setup is reproducible across real-robot runs.

Made-with: Cursor

File: ros2/lerobot_teleoperator_devices/lerobot_teleoperator_devices/processors/_cache/panda_resolved.urdf (robot description, URDF)
Before this commit: robot panda, 12 links, 11 joints
Links:
- link panda_hand: geometry collision mesh filename=/home/cihan/lerobot-ros-agent/ros2/isaac_franka_moveit_perc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; visual mesh filename=/home/cihan/lerobot-ros-agent/ros2/isaac_franka_moveit_perc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
- link panda_leftfinger: geometry collision mesh filename=/home/cihan/lerobot-ros-agent/ros2/isaac_franka_moveit_perc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; visual mesh filename=/home/cihan/lerobot-ros-agent/ros2/isaac_franka_moveit_perc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
- link panda_link0: geometry collision mesh filename=/home/cihan/lerobot-ros-agent/ros2/isaac_franka_moveit_perc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; visual mesh filename=/home/cihan/lerobot-ros-agent/ros2/isaac_franka_moveit_perc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
- link panda_link1: geometry collision mesh filename=/home/cihan/lerobot-ros-agent/ros2/isaac_franka_moveit_perc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; visual mesh filename=/home/cihan/lerobot-ros-agent/ros2/isaac_franka_moveit_perc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
- link panda_link2: geometry collision mesh filename=/home/cihan/lerobot-ros-agent/ros2/isaac_franka_moveit_perc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; visual mesh filename=/home/cihan/lerobot-ros-agent/ros2/isaac_franka_moveit_perc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
- link panda_link3: geometry collision mesh filename=/home/cihan/lerobot-ros-agent/ros2/isaac_franka_moveit_perc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; visual mesh filename=/home/cihan/lerobot-ros-agent/ros2/isaac_franka_moveit_perc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
- link panda_link4: geometry collision mesh filename=/home/cihan/lerobot-ros-agent/ros2/isaac_franka_moveit_perc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; visual mesh filename=/home/cihan/lerobot-ros-agent/ros2/isaac_franka_moveit_perc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
- link panda_link5: geometry collision mesh filename=/home/cihan/lerobot-ros-agent/ros2/isaac_franka_moveit_perc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; visual mesh filename=/home/cihan/lerobot-ros-agent/ros2/isaac_franka_moveit_perc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
- link panda_link6: geometry collision mesh filename=/home/cihan/lerobot-ros-agent/ros2/isaac_franka_moveit_perc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; visual mesh filename=/home/cihan/lerobot-ros-agent/ros2/isaac_franka_moveit_perc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
- link panda_link7: geometry collision mesh filename=/home/cihan/lerobot-ros-agent/ros2/isaac_franka_moveit_perc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; visual mesh filename=/home/cihan/lerobot-ros-agent/ros2/isaac_franka_moveit_perc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
- link panda_rightfinger: geometry collision mesh filename=/home/cihan/lerobot-ros-agent/ros2/isaac_franka_moveit_perc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; visual mesh filename=/home/cihan/lerobot-ros-agent/ros2/isaac_franka_moveit_perc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
